Commit message: endret gitignore

File: seabotics_ws/install/share/hugr_description/urdf/parts/sensors.xacro (robot description, xacro)
@@ -1,20 +1 @@
-<?xml version="1.0"?>
-<xacro:macro xmlns:xacro="http://www.ros.org/wiki/xacro"
-             name="add_sensors" params="">
-  <link name="imu_link">
-    <visual><origin xyz="0 0 0.25"/><geometry><box size="0.05 0.05 0.02"/></geometry></visual>
-  </link>
-  <joint name="imu_joint" type="fixed">
-    <parent link="base_link"/><child link="imu_link"/><origin xyz="0 0 0.25"/>
-  </joint>
-  <link name="oakd_frame">
-    <visual><origin xyz="0.4 0 0.15"/><geometry><box size="0.06 0.06 0.03"/></geometry></visual>
-  </link>
-  <joint name="oakd_joint" type="fixed">
-    <parent link="base_link"/><child link="oakd_frame"/><origin xyz="0.4 0 0.15"/>
-  </joint>
-  <link name="oakd_optical_frame"/>
-  <joint name="oakd_optical_joint" type="fixed">
-    <parent link="oakd_frame"/><child link="oakd_optical_frame"/>
-  </joint>
-</xacro:macro>
+/home/isak/seabotics_ws/Hugr_Primus/seabotics_ws/src/hugr_description/urdf/parts/sensors.xacro

File: seabotics_ws/install/share/hugr_description/urdf/parts/thrusters.xacro (robot description, xacro)
@@ -1,43 +1 @@
-<?xml version="1.0"?>
-<robot name="thruster_parts" xmlns:xacro="http://www.ros.org/wiki/xacro">
-  <material name="mat_thruster"><color rgba="0.2 0.2 0.3 1.0"/></material>
-  <!-- axis: 'x' (default), 'y', or 'z'.  Cylinder is Z-aligned by default in URDF. -->
-  <xacro:macro name="thruster"
-               params="name parent
-                       xyz:='0 0 0'
-                       axis:='x'
-                       diameter:=0.08
-                       length:=0.12
-                       mass:=0.8">
-    <link name="${name}_link">
-      <visual>
-        <origin xyz="0 0 0" rpy="0 0 0"/>
-        <geometry><cylinder radius="${diameter/2.0}" length="${length}"/></geometry>
-        <material name="mat_thruster"/>
-      </visual>
-      <collision>
-        <origin xyz="0 0 0" rpy="0 0 0"/>
-        <geometry><cylinder radius="${diameter/2.0}" length="${length}"/></geometry>
-      </collision>
-      <inertial>
-        <origin xyz="0 0 0" rpy="0 0 0"/>
-        <mass value="${mass}"/>
-        <!-- Cylinder inertia (axis along Z) -->
-        <inertia ixx="${(mass*(3*(diameter/2.0)*(diameter/2.0)+length*length))/12.0}"
-                 iyy="${(mass*(3*(diameter/2.0)*(diameter/2.0)+length*length))/12.0}"
-                 izz="${0.5*mass*(diameter/2.0)*(diameter/2.0)}"
-                 ixy="0" ixz="0" iyz="0"/>
-      </inertial>
-    </link>
-    <!-- Compute orientation so the cylinder aligns with requested axis -->
-    <!-- Orientér sylinder (URDF sylinder peker langs Z som standard) -->
-    <xacro:property name="thr_roll"  value="${ (-pi/2.0) if axis == 'y' else 0.0 }"/>
-    <xacro:property name="thr_pitch" value="${ ( pi/2.0) if axis == 'x' else 0.0 }"/>
-    <xacro:property name="thr_yaw"   value="${ 0.0 }"/>
-    <joint name="${name}_joint" type="fixed">
-      <parent link="${parent}"/>
-      <child  link="${name}_link"/>
-      <origin xyz="${xyz}" rpy="${thr_roll} ${thr_pitch} ${thr_yaw}"/>
-    </joint>
-  </xacro:macro>
-</robot>
+/home/isak/seabotics_ws/Hugr_Primus/seabotics_ws/src/hugr_description/urdf/parts/thrusters.xacro

File: seabotics_ws/install/share/hugr_description/urdf/parts/trimaran_hull.xacro (robot description, xacro)
@@ -1,105 +1 @@
-<?xml version="1.0"?>
-<robot name="trimaran_parts" xmlns:xacro="http://www.ros.org/wiki/xacro">
-  <xacro:macro name="trimaran_hull"
-               params="mass_total:=65.0 L:=1.80 W:=0.40 H:=0.20 outr_len:=1.60 outr_diam:=0.12 beam_thick:=0.05 outr_y:=0.45">
-    <!-- farger -->
-    <material name="mat_white"><color rgba="0.9 0.9 0.9 1.0"/></material>
-    <material name="mat_grey"><color rgba="0.5 0.5 0.5 1.0"/></material>
-    <!-- hjelpe-makroer for inerti -->
-    <xacro:macro name="box_inertia" params="m sx sy sz">
-      <inertial>
-        <origin xyz="0 0 0" rpy="0 0 0"/>
-        <mass value="${m}"/>
-        <inertia ixx="${m*(sy*sy+sz*sz)/12.0}"
-                 iyy="${m*(sx*sx+sz*sz)/12.0}"
-                 izz="${m*(sx*sx+sy*sy)/12.0}"
-                 ixy="0" ixz="0" iyz="0"/>
-      </inertial>
-    </xacro:macro>
-    <xacro:macro name="cyl_x_inertia" params="m r l">
-      <inertial>
-        <origin xyz="0 0 0" rpy="0 0 0"/>
-        <mass value="${m}"/>
-        <inertia ixx="${0.5*m*r*r}"
-                 iyy="${(m*(3*r*r + l*l))/12.0}"
-                 izz="${(m*(3*r*r + l*l))/12.0}"
-                 ixy="0" ixz="0" iyz="0"/>
-      </inertial>
-    </xacro:macro>
-    <!-- hovedskrog (boks) -->
-    <link name="base_link">
-      <visual>
-        <origin xyz="0 0 ${H/2.0}" rpy="0 0 0"/>
-        <geometry><box size="${L} ${W} ${H}"/></geometry>
-        <material name="mat_white"/>
-      </visual>
-      <collision>
-        <origin xyz="0 0 ${H/2.0}" rpy="0 0 0"/>
-        <geometry><box size="${L} ${W} ${H}"/></geometry>
-      </collision>
-      <xacro:box_inertia m="${mass_total*0.7}" sx="${L}" sy="${W}" sz="${H}"/>
-    </link>
-    <!-- tverrbjelker -->
-    <link name="beam_front">
-      <visual>
-        <origin xyz="${-L/3} 0 ${H/2.0}" rpy="0 0 0"/>
-        <geometry><box size="${beam_thick} ${2*outr_y} ${beam_thick}"/></geometry>
-        <material name="mat_grey"/>
-      </visual>
-      <collision>
-        <origin xyz="${-L/3} 0 ${H/2.0}" rpy="0 0 0"/>
-        <geometry><box size="${beam_thick} ${2*outr_y} ${beam_thick}"/></geometry>
-      </collision>
-      <xacro:box_inertia m="${mass_total*0.05}" sx="${beam_thick}" sy="${2*outr_y}" sz="${beam_thick}"/>
-    </link>
-    <joint name="beam_front_joint" type="fixed">
-      <parent link="base_link"/><child link="beam_front"/>
-    </joint>
-    <link name="beam_rear">
-      <visual>
-        <origin xyz="${L/3} 0 ${H/2.0}" rpy="0 0 0"/>
-        <geometry><box size="${beam_thick} ${2*outr_y} ${beam_thick}"/></geometry>
-        <material name="mat_grey"/>
-      </visual>
-      <collision>
-        <origin xyz="${L/3} 0 ${H/2.0}" rpy="0 0 0"/>
-        <geometry><box size="${beam_thick} ${2*outr_y} ${beam_thick}"/></geometry>
-      </collision>
-      <xacro:box_inertia m="${mass_total*0.05}" sx="${beam_thick}" sy="${2*outr_y}" sz="${beam_thick}"/>
-    </link>
-    <joint name="beam_rear_joint" type="fixed">
-      <parent link="base_link"/><child link="beam_rear"/>
-    </joint>
-    <!-- sidepæler -->
-    <link name="outrigger_left">
-      <visual>
-        <origin xyz="0 ${outr_y} ${outr_diam/2.0}" rpy="0 ${pi/2} 0"/>
-        <geometry><cylinder radius="${outr_diam/2.0}" length="${outr_len}"/></geometry>
-        <material name="mat_white"/>
-      </visual>
-      <collision>
-        <origin xyz="0 ${outr_y} ${outr_diam/2.0}" rpy="0 ${pi/2} 0"/>
-        <geometry><cylinder radius="${outr_diam/2.0}" length="${outr_len}"/></geometry>
-      </collision>
-      <xacro:cyl_x_inertia m="${mass_total*0.125}" r="${outr_diam/2.0}" l="${outr_len}"/>
-    </link>
-    <joint name="outrigger_left_joint" type="fixed">
-      <parent link="base_link"/><child link="outrigger_left"/>
-    </joint>
-    <link name="outrigger_right">
-      <visual>
-        <origin xyz="0 ${-outr_y} ${outr_diam/2.0}" rpy="0 ${pi/2} 0"/>
-        <geometry><cylinder radius="${outr_diam/2.0}" length="${outr_len}"/></geometry>
-        <material name="mat_white"/>
-      </visual>
-      <collision>
-        <origin xyz="0 ${-outr_y} ${outr_diam/2.0}" rpy="0 ${pi/2} 0"/>
-        <geometry><cylinder radius="${outr_diam/2.0}" length="${outr_len}"/></geometry>
-      </collision>
-      <xacro:cyl_x_inertia m="${mass_total*0.125}" r="${outr_diam/2.0}" l="${outr_len}"/>
-    </link>
-    <joint name="outrigger_right_joint" type="fixed">
-      <parent link="base_link"/><child link="outrigger_right"/>
-    </joint>
-  </xacro:macro>
-</robot>
+/home/isak/seabotics_ws/Hugr_Primus/seabotics_ws/src/hugr_description/urdf/parts/trimaran_hull.xacro
